Commit message: Slam and camera

File: src/lampo_description/urdf/system.urdf.xacro (robot description, xacro)
@@ -55,5 +55,5 @@
   <xacro:if value="$(arg mm)">
     <xacro:fake_camera prefix="$(arg prefix)" parent="$(arg prefix)tool0">
-      <origin xyz="0 0 0.05" rpy="0 0 0" />
+      <origin xyz="0 0 0.05" rpy="1.57 -1.57 1.57" />
     </xacro:fake_camera>
   </xacro:if>
@@ -83,5 +83,5 @@
         <joint_name>$(arg prefix_rc)/shoulder_pan_joint</joint_name>
         <topic>$(arg prefix_rc)/shoulder_pan_joint</topic>
-        <p_gain>2000</p_gain>
+        <p_gain>5000</p_gain>
         <i_gain>0.1</i_gain>
         <d_gain>200.00</d_gain>
@@ -99,5 +99,5 @@
         <joint_name>$(arg prefix_rc)/shoulder_lift_joint</joint_name>
         <topic>$(arg prefix_rc)/shoulder_lift_joint</topic>
-        <p_gain>2000</p_gain>
+        <p_gain>10000</p_gain>
         <i_gain>0.1</i_gain>
         <d_gain>200.00</d_gain>
@@ -115,5 +115,5 @@
         <joint_name>$(arg prefix_rc)/elbow_joint</joint_name>
         <topic>$(arg prefix_rc)/elbow_joint</topic>
-        <p_gain>2000</p_gain>
+        <p_gain>10000</p_gain>
         <i_gain>0.1</i_gain>
         <d_gain>200.00</d_gain>
@@ -163,5 +163,5 @@
         <joint_name>$(arg prefix_rc)/wrist_3_joint</joint_name>
         <topic>$(arg prefix_rc)/wrist_3_joint</topic>
-        <p_gain>2000</p_gain>
+        <p_gain>0</p_gain>
         <i_gain>0.1</i_gain>
         <d_gain>200.00</d_gain>
@@ -183,5 +183,5 @@
       <hardware>
           <plugin>topic_based_ros2_control/TopicBasedSystem</plugin>
-          <!-- <plugin>gazebo_ros2_control/GazeboSystem</plugin> -->
+          <!-- <plugin>gz_ros2_control/GazeboSimSystem</plugin> -->
           <param name="joint_commands_topic">joint_commands</param>
           <param name="joint_states_topic">jnt_gz</param>
